Commit message: update

File: src/galbot_s1_v1_description/urdf/galbot_S1_V1_with_GE10301.urdf.xacro (robot description, xacro)
@@ -2206,3 +2206,73 @@
   </actuator>
 </transmission>
+<!-- <transmission name="left_arm_joint1_trans">
+  <type>transmission_interface/SimpleTransmission</type>
+  <joint name="left_arm_joint1">
+    <hardwareInterface>hardware_interface/PositionJointInterface</hardwareInterface>
+  </joint>
+  <actuator name="left_arm_joint1_motor">
+    <hardwareInterface>hardware_interface/PositionJointInterface</hardwareInterface>
+    <mechanicalReduction>1</mechanicalReduction>
+  </actuator>
+</transmission>
+<transmission name="left_arm_joint2_trans">
+  <type>transmission_interface/SimpleTransmission</type>
+  <joint name="left_arm_joint2">
+    <hardwareInterface>hardware_interface/PositionJointInterface</hardwareInterface>
+  </joint>
+  <actuator name="left_arm_joint2_motor">
+    <hardwareInterface>hardware_interface/PositionJointInterface</hardwareInterface>
+    <mechanicalReduction>1</mechanicalReduction>
+  </actuator>
+</transmission>
+<transmission name="left_arm_joint3_trans">
+  <type>transmission_interface/SimpleTransmission</type>
+  <joint name="left_arm_joint3">
+    <hardwareInterface>hardware_interface/PositionJointInterface</hardwareInterface>
+  </joint>
+  <actuator name="left_arm_joint3_motor">
+    <hardwareInterface>hardware_interface/PositionJointInterface</hardwareInterface>
+    <mechanicalReduction>1</mechanicalReduction>
+  </actuator>
+</transmission>
+<transmission name="left_arm_joint4_trans">
+  <type>transmission_interface/SimpleTransmission</type>
+  <joint name="left_arm_joint4">
+    <hardwareInterface>hardware_interface/PositionJointInterface</hardwareInterface>
+  </joint>
+  <actuator name="left_arm_joint4_motor">
+    <hardwareInterface>hardware_interface/PositionJointInterface</hardwareInterface>
+    <mechanicalReduction>1</mechanicalReduction>
+  </actuator>
+</transmission>
+<transmission name="left_arm_joint5_trans">
+  <type>transmission_interface/SimpleTransmission</type>
+  <joint name="left_arm_joint5">
+    <hardwareInterface>hardware_interface/PositionJointInterface</hardwareInterface>
+  </joint>
+  <actuator name="left_arm_joint5_motor">
+    <hardwareInterface>hardware_interface/PositionJointInterface</hardwareInterface>
+    <mechanicalReduction>1</mechanicalReduction>
+  </actuator>
+</transmission>
+<transmission name="left_arm_joint6_trans">
+  <type>transmission_interface/SimpleTransmission</type>
+  <joint name="left_arm_joint6">
+    <hardwareInterface>hardware_interface/PositionJointInterface</hardwareInterface>
+  </joint>
+  <actuator name="left_arm_joint6_motor">
+    <hardwareInterface>hardware_interface/PositionJointInterface</hardwareInterface>
+    <mechanicalReduction>1</mechanicalReduction>
+  </actuator>
+</transmission>
+<transmission name="left_arm_joint7_trans">
+  <type>transmission_interface/SimpleTransmission</type>
+  <joint name="left_arm_joint7">
+    <hardwareInterface>hardware_interface/PositionJointInterface</hardwareInterface>
+  </joint>
+  <actuator name="left_arm_joint7_motor">
+    <hardwareInterface>hardware_interface/PositionJointInterface</hardwareInterface>
+    <mechanicalReduction>1</mechanicalReduction>
+  </actuator>
+</transmission> -->
 </robot>

Commit message: update arm

File: src/galbot_s1_v1_description/urdf/galbot_S1_V1_with_GE10301.urdf.xacro (robot description, xacro)
@@ -1001,5 +1001,5 @@
   <joint
     name="left_arm_joint1"
-    type="fixed">
+    type="revolute">
     <origin
       xyz="0 0 0"
@@ -1059,5 +1059,5 @@
   <joint
     name="left_arm_joint2"
-    type="fixed">
+    type="revolute">
     <origin
       xyz="0 0 0"
@@ -1117,5 +1117,5 @@
   <joint
     name="left_arm_joint3"
-    type="fixed">
+    type="revolute">
     <origin
       xyz="0 0.49 0"
@@ -1175,5 +1175,5 @@
   <joint
     name="left_arm_joint4"
-    type="fixed">
+    type="revolute">
     <origin
       xyz="0 0 0"
@@ -1233,5 +1233,5 @@
   <joint
     name="left_arm_joint5"
-    type="fixed">
+    type="revolute">
     <origin
       xyz="0 -0.4307 4.6056E-05"
@@ -1291,5 +1291,5 @@
   <joint
     name="left_arm_joint6"
-    type="fixed">
+    type="revolute">
     <origin
       xyz="0 0 0"
@@ -1349,5 +1349,5 @@
   <joint
     name="left_arm_joint7"
-    type="fixed">
+    type="revolute">
     <origin
       xyz="0 0 0"
@@ -1452,5 +1452,5 @@
   <joint
     name="right_arm_joint1"
-    type="fixed">
+    type="revolute">
     <origin
       xyz="0 0 0"
@@ -1510,5 +1510,5 @@
   <joint
     name="right_arm_joint2"
-    type="fixed">
+    type="revolute">
     <origin
       xyz="0 0 0"
@@ -1568,5 +1568,5 @@
   <joint
     name="right_arm_joint3"
-    type="fixed">
+    type="revolute">
     <origin
       xyz="0 -0.49 0"
@@ -1626,5 +1626,5 @@
   <joint
     name="right_arm_joint4"
-    type="fixed">
+    type="revolute">
     <origin
       xyz="0 0 0"
@@ -1684,5 +1684,5 @@
   <joint
     name="right_arm_joint5"
-    type="fixed">
+    type="revolute">
     <origin
       xyz="0 0.43072 4.6056E-05"
@@ -1742,5 +1742,5 @@
   <joint
     name="right_arm_joint6"
-    type="fixed">
+    type="revolute">
     <origin
       xyz="0 0 0"
@@ -1800,5 +1800,5 @@
   <joint
     name="right_arm_joint7"
-    type="fixed">
+    type="revolute">
     <origin
       xyz="0 0 0"
@@ -2206,5 +2206,5 @@
   </actuator>
 </transmission>
-<!-- <transmission name="left_arm_joint1_trans">
+<transmission name="left_arm_joint1_trans">
   <type>transmission_interface/SimpleTransmission</type>
   <joint name="left_arm_joint1">
@@ -2275,4 +2275,74 @@
     <mechanicalReduction>1</mechanicalReduction>
   </actuator>
-</transmission> -->
+</transmission>
+<transmission name="right_arm_joint1_trans">
+  <type>transmission_interface/SimpleTransmission</type>
+  <joint name="right_arm_joint1">
+    <hardwareInterface>hardware_interface/PositionJointInterface</hardwareInterface>
+  </joint>
+  <actuator name="right_arm_joint1_motor">
+    <hardwareInterface>hardware_interface/PositionJointInterface</hardwareInterface>
+    <mechanicalReduction>1</mechanicalReduction>
+  </actuator>
+</transmission>
+<transmission name="right_arm_joint2_trans">
+  <type>transmission_interface/SimpleTransmission</type>
+  <joint name="right_arm_joint2">
+    <hardwareInterface>hardware_interface/PositionJointInterface</hardwareInterface>
+  </joint>
+  <actuator name="right_arm_joint2_motor">
+    <hardwareInterface>hardware_interface/PositionJointInterface</hardwareInterface>
+    <mechanicalReduction>1</mechanicalReduction>
+  </actuator>
+</transmission>
+<transmission name="right_arm_joint3_trans">
+  <type>transmission_interface/SimpleTransmission</type>
+  <joint name="right_arm_joint3">
+    <hardwareInterface>hardware_interface/PositionJointInterface</hardwareInterface>
+  </joint>
+  <actuator name="right_arm_joint3_motor">
+    <hardwareInterface>hardware_interface/PositionJointInterface</hardwareInterface>
+    <mechanicalReduction>1</mechanicalReduction>
+  </actuator>
+</transmission>
+<transmission name="right_arm_joint4_trans">
+  <type>transmission_interface/SimpleTransmission</type>
+  <joint name="right_arm_joint4">
+    <hardwareInterface>hardware_interface/PositionJointInterface</hardwareInterface>
+  </joint>
+  <actuator name="right_arm_joint4_motor">
+    <hardwareInterface>hardware_interface/PositionJointInterface</hardwareInterface>
+    <mechanicalReduction>1</mechanicalReduction>
+  </actuator>
+</transmission>
+<transmission name="right_arm_joint5_trans">
+  <type>transmission_interface/SimpleTransmission</type>
+  <joint name="right_arm_joint5">
+    <hardwareInterface>hardware_interface/PositionJointInterface</hardwareInterface>
+  </joint>
+  <actuator name="right_arm_joint5_motor">
+    <hardwareInterface>hardware_interface/PositionJointInterface</hardwareInterface>
+    <mechanicalReduction>1</mechanicalReduction>
+  </actuator>
+</transmission>
+<transmission name="right_arm_joint6_trans">
+  <type>transmission_interface/SimpleTransmission</type>
+  <joint name="right_arm_joint6">
+    <hardwareInterface>hardware_interface/PositionJointInterface</hardwareInterface>
+  </joint>
+  <actuator name="right_arm_joint6_motor">
+    <hardwareInterface>hardware_interface/PositionJointInterface</hardwareInterface>
+    <mechanicalReduction>1</mechanicalReduction>
+  </actuator>
+</transmission>
+<transmission name="right_arm_joint7_trans">
+  <type>transmission_interface/SimpleTransmission</type>
+  <joint name="right_arm_joint7">
+    <hardwareInterface>hardware_interface/PositionJointInterface</hardwareInterface>
+  </joint>
+  <actuator name="right_arm_joint7_motor">
+    <hardwareInterface>hardware_interface/PositionJointInterface</hardwareInterface>
+    <mechanicalReduction>1</mechanicalReduction>
+  </actuator>
+</transmission>
 </robot>
